File: hardware/StevePico6502/StevePico6592.kicad_pcb (KiCad board)
At the start: 2 copper layers, 128.4 x 124 mm, 32 parts, among them J1 Conn_01x16, J2 Conn_01x16, J3 Conn_02x16_Odd_Even, J4 Conn_01x02_Pin, J5 Conn_01x02_Pin, J6 Conn_02x11_Odd_Even, J7 Conn_01x02_Pin, SW1 SW_Push, U1 W65C02S, U2 28C256, U3 CY62256-70PC, U4 W65C22S, U5 74HC00, X1 CXO_DIP14

Commit message: V091723 before fab
Parts:
- added C11: 1uF, Capacitor_THT:C_Disc_D3.4mm_W2.1mm_P2.50mm, F.Cu at (88.3, 92.9)
- added C13: 20pF, Capacitor_THT:C_Disc_D3.4mm_W2.1mm_P2.50mm, F.Cu at (140.9, 109.4)
- added D2: SB140, Diode_THT:D_DO-41_SOD81_P10.16mm_Horizontal, F.Cu at (82.8, 76.1)
- added J10: FTDI Power, Connector_PinHeader_2.54mm:PinHeader_1x02_P2.54mm_Vertical, F.Cu at (149.8, 109.9)
- added J8: CLK SELECT, Connector_PinHeader_2.54mm:PinHeader_1x02_P2.54mm_Vertical, F.Cu at (159.8, 113.2)
- added J9: FTDI Connector, Connector_PinHeader_2.54mm:PinHeader_1x06_P2.54mm_Vertical, F.Cu at (159.8, 104.3)
- added R4: 1m, Resistor_THT:R_Axial_DIN0207_L6.3mm_D2.5mm_P7.62mm_Horizontal, F.Cu at (147.3, 105.0)
- added U6: W6551, Package_DIP:DIP-28_W15.24mm, F.Cu at (92.6, 99.3)
- added Y1: 1.843, Crystal:Crystal_HC52-8mm_Vertical, F.Cu at (141.3, 103.0)
- J1: value Conn_01x16 -> GPIOB
- J2: value Conn_01x16 -> GPIOA
- J4: value Conn_01x02_Pin -> ROM SELECT
- J5: value Conn_01x02_Pin -> RAM SELECT
- J6: value Conn_02x11_Odd_Even -> Expansion
- J7: value Conn_01x02_Pin -> IO SELECT
- RV1: footprint Potentiometer_THT:Potentiometer_Bourns_3296W_Vertical -> Potentiometer_THT:Potentiometer_Piher_PT-6-V_Vertical
- moved J6 94.4 mm to (162.3, 148.0), turned to 180 degrees
- moved J3 68.8 mm to (182.2, 111.8), turned to 0 degrees
- moved C3 52.4 mm to (182.5, 153.9), turned to 0 degrees
- moved J5 49.6 mm to (119.4, 112.4), turned to 180 degrees
- moved J4 48.4 mm to (123.2, 112.4), turned to 180 degrees
- moved J7 47.9 mm to (127.0, 112.4), turned to 180 degrees
- moved J2 46.8 mm to (165.7, 40.6)
- moved C5 46.8 mm to (165.7, 84.8)
- moved C1 27.5 mm to (70.5, 114.3)
- moved C9 25.7 mm to (91.9, 109.8)
- moved U5 25.7 mm to (96.5, 112.4)
- moved C4 19.5 mm to (182.9, 84.8)
- moved J1 19.5 mm to (182.9, 40.6)
- moved X1 11.1 mm to (75.6, 96.5), turned to -90 degrees
- moved C2 7.75 mm to (62.9, 101.6), turned to -90 degrees
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Connections:
- X1 pad 8: /CLK -> /CLK_INT
Routing:
- net /~{IOSEL}: track 108.0 -> 230.4 mm, vias 0 -> 1
- net /A7: track 135.2 -> 230.5 mm
- net /CLK: track 203.2 -> 296.3 mm, vias 2 -> 0
- net VCC: track 474.4 -> 564.8 mm, vias 0 -> 1
- net /A8: track 149.7 -> 238.0 mm
- net /CLK_INT: track 0.00 -> 86.0 mm
- net /A0: track 156.8 -> 240.0 mm
- net GND: track 460.1 -> 542.1 mm, vias 1 -> 2
- net /A5: track 124.6 -> 204.7 mm, vias 1 -> 2
- net /~{ROMSEL}: track 167.3 -> 90.5 mm, vias 1 -> 0
- net /~{ROMSEL_INT}: track 105.0 -> 32.9 mm, vias 3 -> 0
- net /~{IOSEL_INT}: track 90.2 -> 18.2 mm
- net /~{RAMSEL_INT}: track 83.8 -> 12.1 mm
- net /D7: track 157.3 -> 227.4 mm
- net /D0: track 129.7 -> 198.9 mm
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Other:
- board size 128.4 x 124 mm -> 145.3 x 124 mm
- board text added: "FTDI Conn"
- board text added: "V0901723"
- board text removed: "V090423"

Commit message: 'V091723'
Parts:
- removed DS1: WC1602A, Display:WC1602A
- removed J4: ROM SELECT, Connector_PinHeader_2.54mm:PinHeader_1x02_P2.54mm_Vertical
- removed J5: RAM SELECT, Connector_PinHeader_2.54mm:PinHeader_1x02_P2.54mm_Vertical
- removed J6: Expansion, Connector_PinHeader_2.54mm:PinHeader_2x11_P2.54mm_Vertical
- removed J7: IO SELECT, Connector_PinHeader_2.54mm:PinHeader_1x02_P2.54mm_Vertical
- removed RV1: 10k, Potentiometer_THT:Potentiometer_Piher_PT-6-V_Vertical
- removed U5: 74HC00, Package_DIP:DIP-14_W7.62mm_Socket_LongPads
- added D3: SB140, Diode_THT:D_DO-41_SOD81_P10.16mm_Horizontal, F.Cu at (159.8, 83.2)
- added U7: GAL16V8, Package_DIP:DIP-20_W7.62mm_Socket_LongPads, F.Cu at (97.9, 112.3)
- J3: value Conn_02x16_Odd_Even -> Conn_02x20_Odd_Even; footprint Connector_PinHeader_2.54mm:PinHeader_2x16_P2.54mm_Vertical -> Connector_PinHeader_2.54mm:PinHeader_2x20_P2.54mm_Vertical
- J8: footprint Connector_PinHeader_2.54mm:PinHeader_1x02_P2.54mm_Vertical -> Connector_PinHeader_2.54mm:PinHeader_1x03_P2.54mm_Vertical
- U6: footprint Package_DIP:DIP-28_W15.24mm -> Package_DIP:DIP-28_W15.24mm_Socket_LongPads
- moved D2 49.5 mm to (132.3, 78.1)
- moved J3 45.8 mm to (137.9, 123.2), turned to 90 degrees
- moved C3 34.2 mm to (190.2, 120.6), turned to -90 degrees
- moved REF** 32.4 mm to (87.6, 126.1)
- moved J8 30.1 mm to (189.7, 110.2), turned to -90 degrees
- moved C1 19.4 mm to (77.5, 96.2), turned to 0 degrees
- moved X1 13.7 mm to (71.2, 109.5), turned to 0 degrees
- moved J10 12.2 mm to (147.8, 97.8), turned to 90 degrees
- moved C13 8.75 mm to (132.5, 107.1)
- moved R4 8.75 mm to (138.8, 102.6)
- moved Y1 8.75 mm to (132.8, 100.7)
- moved J9 1.50 mm to (159.8, 102.8)
- moved C4 1.19 mm to (182.9, 83.6)
- moved C5 1.19 mm to (165.7, 83.6)
- moved J1 1.19 mm to (182.9, 39.5)
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Connections:
- J3 pad 30: VCC -> /~{ROMSEL}
- J3 pad 32: GND -> /6522SEL
- J8 pad 1: /CLK -> /CLK_ALT
- J8 pad 2: /CLK_INT -> /CLK
- U4 pad 21: /~{IRQ} -> Net-(D3-K)
- U4 pad 24: /A13 -> /6522SEL
- U6 pad 2: /A12 -> /ACIASEL
- U6 pad 26: /~{IRQ} -> Net-(D2-K)
Routing:
- net /~{ROMSEL}: track 90.5 -> 255.3 mm, vias 0 -> 1
- net /6522SEL: track 0.00 -> 121.9 mm, vias 0 -> 2
- net /GPIOB2: track 180.4 -> 61.5 mm, vias 0 -> 1
- net /GPIOB0: track 155.6 -> 53.8 mm
- net /ACIASEL: track 0.00 -> 100.8 mm, vias 0 -> 1
- net /GPIOB1: track 148.6 -> 53.8 mm
- net VCC: track 564.8 -> 481.1 mm
- net /GPIOB3: track 136.5 -> 53.8 mm, vias 1 -> 0
- net /GPIOB5: track 135.1 -> 53.8 mm, vias 1 -> 0
- net /GPIOA5: track 106.5 -> 28.3 mm
- net /GPIOB4: track 130.9 -> 53.8 mm
- net /LCD_D0: track 73.8 -> 0.00 mm, vias 1 -> 0
- net /LCD_RS: track 73.0 -> 0.00 mm
- net /GPIOA6: track 102.0 -> 29.2 mm
- net /LCD_D1: track 70.2 -> 0.00 mm, vias 1 -> 0
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Other:
- board size 145.3 x 124 mm -> 145.3 x 101.1 mm
- board text removed: "Connect to use internal glue logic"
- board text removed: "Jumper to connect LCD to GPIOB and the 3 highest bits of GPIOA"
- board text removed: "LCD Enable"
