File: hardware/StevePico6502/StevePico6592.kicad_sch (KiCad schematic)
At the start: 28 parts, among them J1 Conn_01x16, J2 Conn_01x16, J3 Conn_02x16_Odd_Even, J6 Conn_02x11_Odd_Even, SW1 SW_Push, U1 W65C02, U2 28C256, U3 CY62256-70PC, U4 W65C22S, U5 74HC00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

Commit message: V090423
Parts:
- added J4, J5, J7: Conn_01x02_Pin, Connector_PinHeader_2.54mm:PinHeader_1x02_P2.54mm_Vertical, symbol Connector:Conn_01x02_Pin
- U1: value W65C02 -> W65C02S
Connections:
- net A14: now also U3.22 (~{OE})
- net GND: now also U2.22 (~{OE}); no longer U3.22 (~{OE})
- net R~{W}: no longer U2.22 (~{OE})
- net ~{IOSEL}: now also J7.1 (Pin_1); no longer U5.8
- net ~{RAMSEL}: now also J5.1 (Pin_1); no longer U5.6
- net ~{ROMSEL}: now also J4.1 (Pin_1); no longer U5.3, U5.4, U5.9
- new net ~{IOSEL_INT}: J7.2 (Pin_2), U5.8
- new net ~{RAMSEL_INT}: J5.2 (Pin_2), U5.6
- new net ~{ROMSEL_INT}: J4.2 (Pin_2), U5.3, U5.4, U5.9
Other:
- moved on the sheet: C1

Commit message: Working on ACIA
Parts:
- added C11, C12: 1uF, Capacitor_THT:C_Disc_D3.4mm_W2.1mm_P2.50mm, symbol Device:C
- added J8: CLK SELECT, Connector_PinHeader_2.54mm:PinHeader_1x02_P2.54mm_Vertical, symbol Connector:Conn_01x02_Pin
- added U6: W6551, symbol 6502:W65C51
- added X2: CXO_DIP14, Oscillator:Oscillator_DIP-14, symbol Oscillator:CXO_DIP14
- J1: value Conn_01x16 -> GPIOB
- J2: value Conn_01x16 -> GPIOA
- J4: value Conn_01x02_Pin -> ROM SELECT
- J5: value Conn_01x02_Pin -> RAM SELECT
- J6: value Conn_02x11_Odd_Even -> Expansion
- J7: value Conn_01x02_Pin -> IO SELECT
Connections:
- net A0: now also U6.13 (RS0)
- net A1: now also U6.14 (RS1)
- net A12: now also U6.2 (CS0)
- net CLK: now also J8.1 (Pin_1), U6.27 (PHI2); no longer X1.8 (OUT)
- net D0: now also U6.18 (D0)
- net D1: now also U6.19 (D1)
- net D2: now also U6.20 (D2)
- net D3: now also U6.21 (D3)
- net D4: now also U6.22 (D4)
- net D5: now also U6.23 (D5)
- net D6: now also U6.24 (D6)
- net D7: now also U6.25 (D7)
- net GND: now also C11.2, C12.2, U6.1 (GND), X2.7 (GND)
- net R~{W}: now also U6.28 (R~{W})
- net VCC: now also C11.1, C12.1, U6.15 (VCC), X2.14 (Vcc)
- net ~{IOSEL}: now also U6.3 (~{CS1})
- net ~{IRQ}: now also U6.26 (~{IRQ})
- net ~{RESET}: now also U6.4 (~{RESET})
- new net CLK_INT: J8.2 (Pin_2), X1.8 (OUT)
- new net RX: U6.12 (RX)
- new net TX: U6.10 (TX)
- new net UART_CLK: U6.6 (XTL1), X2.8 (OUT)
- no-connect marks 15 -> 22
Other:
- note added: "RAM"
- note added: "ROM"
- moved on the sheet: C10, C4, C5, C6, C7, C8, C9, D1, DS1, J1, J2, J4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

Commit message: V091723 before fab
Parts:
- removed C11, C12: 1uF, Capacitor_THT:C_Disc_D3.4mm_W2.1mm_P2.50mm, symbol Device:C
- removed X2: CXO_DIP14, Oscillator:Oscillator_DIP-14, symbol Oscillator:CXO_DIP14
- added C13: 20pF, Capacitor_THT:C_Disc_D3.4mm_W2.1mm_P2.50mm, symbol Device:C
- added D2: SB140, Diode_THT:D_DO-41_SOD81_P10.16mm_Horizontal, symbol Diode:SB140
- added J10: FTDI Power, Connector_PinHeader_2.54mm:PinHeader_1x02_P2.54mm_Vertical, symbol Connector:Conn_01x02_Pin
- added J9: FTDI Connector, Connector_PinHeader_2.54mm:PinHeader_1x06_P2.54mm_Vertical, symbol Connector:Conn_01x06_Pin
- added R4: 1m, Resistor_THT:R_Axial_DIN0207_L6.3mm_D2.5mm_P7.62mm_Horizontal, symbol Device:R
- added Y1: 1.843, Crystal:Crystal_HC52-8mm_Vertical, symbol Device:Crystal
- RV1: footprint Potentiometer_THT:Potentiometer_Bourns_3296W_Vertical -> Potentiometer_THT:Potentiometer_Piher_PT-6-V_Vertical
Connections:
- net GND: now also U6.9 (~{CTS}), C13.2, J9.1 (Pin_1), J9.6 (Pin_6)
- net RX: now also J9.4 (Pin_4)
- net TX: now also J9.5 (Pin_5)
- net VCC: now also J10.2 (Pin_2)
- net ~{IRQ}: now also D2.2 (A); no longer U6.26 (~{IRQ})
- net at U6.11 (~{DTR}): now also U6.16 (~{DCD}), U6.17 (~{DSR})
- net at U6.7 (XTL2): now also R4.1, Y1.1
- net RTS: now reaches U6.8 (~{RTS})
- net RTS: now also J9.2 (Pin_2)
- net UART_CLK: no longer names the net of U6.6 (XTL1)
- net UART_CLK: now also C13.1, R4.2, Y1.2
- new net: D2.1 (K), U6.26 (~{IRQ})
- new net: J10.1 (Pin_1), J9.3 (Pin_3)
- no-connect marks 22 -> 16
Other:
- moved on the sheet: C1, C10, C3, C7, C9, D1, DS1, J3, J4, J6, R1, R2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

Commit message: 'V091723'
Parts:
- removed DS1: WC1602A, Display:WC1602A, symbol Display_Character:WC1602A
- removed J3: Conn_02x16_Odd_Even, Connector_PinHeader_2.54mm:PinHeader_2x16_P2.54mm_Vertical, symbol Connector_Generic:Conn_02x16_Odd_Even
- removed J4: ROM SELECT, Connector_PinHeader_2.54mm:PinHeader_1x02_P2.54mm_Vertical, symbol Connector:Conn_01x02_Pin
- removed J5: RAM SELECT, Connector_PinHeader_2.54mm:PinHeader_1x02_P2.54mm_Vertical, symbol Connector:Conn_01x02_Pin
- removed J6: Expansion, Connector_PinHeader_2.54mm:PinHeader_2x11_P2.54mm_Vertical, symbol Connector_Generic:Conn_02x11_Odd_Even
- removed J7: IO SELECT, Connector_PinHeader_2.54mm:PinHeader_1x02_P2.54mm_Vertical, symbol Connector:Conn_01x02_Pin
- removed RV1: 10k, Potentiometer_THT:Potentiometer_Piher_PT-6-V_Vertical, symbol Device:R_Potentiometer
- removed U5: 74HC00, Package_DIP:DIP-14_W7.62mm_Socket_LongPads, symbol 74xx:74HC00
- added D3: SB140, Diode_THT:D_DO-41_SOD81_P10.16mm_Horizontal, symbol Diode:SB140
- added J3: Conn_02x20_Odd_Even, Connector_PinHeader_2.54mm:PinHeader_2x20_P2.54mm_Vertical, symbol Connector_Generic:Conn_02x20_Odd_Even
- added U7: GAL16V8, Package_DIP:DIP-20_W7.62mm_Socket_LongPads, symbol Logic_Programmable:GAL16V8
- J8: footprint Connector_PinHeader_2.54mm:PinHeader_1x02_P2.54mm_Vertical -> Connector_PinHeader_2.54mm:PinHeader_1x03_P2.54mm_Vertical; symbol Connector:Conn_01x02_Pin -> Connector:Conn_01x03_Pin
- U6: footprint (none) -> Package_DIP:DIP-28_W15.24mm_Socket_LongPads
Connections:
- net A0: now also J3.1 (Pin_1)
- net A1: now also J3.3 (Pin_3)
- net A10: now also J3.21 (Pin_21), U7.6 (I6)
- net A11: now also J3.23 (Pin_23), U7.5 (I5)
- net A12: now also J3.25 (Pin_25), U7.4 (I4); no longer U6.2 (CS0)
- net A13: now also J3.27 (Pin_27), U7.3 (I3); no longer U4.24 (CS1)
- net A14: now also J3.29 (Pin_29), U7.2 (I2)
- net A15: now also J3.31 (Pin_31), U7.1 (I1/CLK)
- net A2: now also J3.5 (Pin_5)
- net A3: now also J3.7 (Pin_7)
- net A4: now also J3.9 (Pin_9)
- net A5: now also J3.11 (Pin_11)
- net A6: now also J3.13 (Pin_13)
- net A7: now also J3.15 (Pin_15)
- net A8: now also J3.17 (Pin_17)
- net A9: now also J3.19 (Pin_19)
- net CLK: now also J8.2 (Pin_2), J3.24 (Pin_24), U7.9 (I9); no longer J8.1 (Pin_1)
- net CLK_INT: now also J8.3 (Pin_3); no longer J8.2 (Pin_2)
- net D0: now also J3.2 (Pin_2)
- net D1: now also J3.4 (Pin_4)
- net D2: now also J3.6 (Pin_6)
- net D3: now also J3.8 (Pin_8)
- net D4: now also J3.10 (Pin_10)
- net D5: now also J3.12 (Pin_12)
- net D6: now also J3.14 (Pin_14)
- net D7: now also J3.16 (Pin_16)
- net GND: now also J3.40 (Pin_40), U7.10 (GND)
- net R~{W}: now also J3.22 (Pin_22), U7.8 (I8)
- net VCC: now also J3.38 (Pin_38), U7.20 (VCC)
- net ~{IOSEL}: now also J3.26 (Pin_26), U7.17 (I03), U7.7 (I7)
- net ~{IRQ}: now also D3.2 (A), J3.20 (Pin_20); no longer U4.21 (~{IRQ})
- net ~{RAMSEL}: now also J3.28 (Pin_28), U7.18 (IO2)
- net ~{RESET}: now also J3.18 (Pin_18)
- net ~{ROMSEL}: now also J3.30 (Pin_30), U7.19 (IO1)
- new net: D3.1 (K), U4.21 (~{IRQ})
- new net 6522SEL: J3.32 (Pin_32), U4.24 (CS1), U7.16 (IO4)
- new net ACIASEL: J3.34 (Pin_34), U6.2 (CS0), U7.15 (IO5)
- new net CLK_ALT: J3.39 (Pin_39), J8.1 (Pin_1)
- no-connect marks 16 -> 22
Other:
- note added: "Address Decode"
- moved on the sheet: D1, R5
